File: hardware/diy_tof_hw/diy_tof_hw.kicad_pcb (KiCad board)
At the start: 4 copper layers, 90 x 100 mm, 83 parts, among them IC1 TDC7200PWR, IC2 TDC7200PWR, IC21 74LVC1G08QW5-7, IC22 LMG1025QDEETQ1, J1 Conn_01x02_Pin, J2 Conn_01x03_Pin, J3 Conn_01x02_Pin, SW1 SW_Nidec_CAS-120A1, SW2 SW_Nidec_CAS-120A1, U1 NUCLEO-F042K6, U2 OPA858xDSG, U3 TLV3501AIDBV, X1 SG-5032CAN

Commit message: [hardware/minor] add value for optic mountings
Signed-off-by: Timon Burkard <burkard.timon@gmail.com>
Parts:
- X2, X3: value ~ -> G061041000
Changed lines of the file:
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@@
 			)
 		)
-		(property "Value" "~"
+		(property "Value" "G061041000"
 			(at 0 1 0)
 			(unlocked yes)
@@
 			)
 		)
-		(property "Value" "~"
+		(property "Value" "G061041000"
 			(at 0 1 0)
 			(unlocked yes)
